Commit message: recovered changes made to panda_moveit_config before fork

File: config/panda_arm.xacro (robot description, xacro)
@@ -18,5 +18,5 @@
       <joint name="panda_joint5" value="0" />
       <joint name="panda_joint6" value="1.571" />
-      <joint name="panda_joint7" value="0.785" />
+      <joint name="panda_joint7" value="-0.785" />
     </group_state>
     <!--END EFFECTOR: Purpose: Represent information about an end effector.-->
@@ -43,4 +43,6 @@
     <disable_collisions link1="panda_link5" link2="panda_link6" reason="Adjacent" />
     <disable_collisions link1="panda_link6" link2="panda_link7" reason="Adjacent" />
+    <disable_collisions link1="panda_link6" link2="panda_link8" reason="Adjacent" />
+    <disable_collisions link1="panda_link7" link2="panda_link8" reason="Adjacent" />
   </xacro:macro>
 </robot>

File: config/panda_arm_hand.srdf.xacro (robot description, xacro)
@@ -35,4 +35,5 @@
   <disable_collisions link1="panda_hand" link2="panda_link6" reason="Never" />
   <disable_collisions link1="panda_hand" link2="panda_link7" reason="Adjacent" />
+  <disable_collisions link1="panda_hand" link2="panda_link8" reason="Adjacent" />
   <disable_collisions link1="panda_leftfinger" link2="panda_link3" reason="Never" />
   <disable_collisions link1="panda_leftfinger" link2="panda_link4" reason="Never" />
